File: nurd-euro-pi.kicad_pcb (KiCad board)
At the start: 2 copper layers, 106.7 x 55.9 mm, 45 parts, among them J1 RPi_GPIO, J2 AudioJack2, J3 AudioJack2, J4 AudioJack2, J5 AudioJack2, J6 AudioJack2, J7 AudioJack2, Q1 2N3904, Q2 2N3904, U1 tl072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

Commit message: Added gate-out
Parts:
- removed C1, C2: 10uF, Capacitor_THT:CP_Radial_D5.0mm_P2.50mm
- removed U4: ICL7660, Package_DIP:DIP-8_W7.62mm_Socket_LongPads
- added J10: AudioJack2, Connector_Audio:Jack_3.5mm_QingPu_WQP-PJ398SM_Vertical_CircularHoles, F.Cu at (31.8, 57.1)
- added J8: Eurorack_Power_16pin_Shrouded, 4ms_Connector:Pins_2x08_2.54mm_TH_EuroPower_Shrouded, F.Cu at (95.2, 66.0)
- added J9: AudioJack2, Connector_Audio:Jack_3.5mm_QingPu_WQP-PJ398SM_Vertical_CircularHoles, F.Cu at (31.8, 77.5)
- added Q3: BC557, Package_TO_SOT_THT:TO-92_Inline, F.Cu at (34.3, 95.2)
- added Q4: BC557, Package_TO_SOT_THT:TO-92_Inline, F.Cu at (27.9, 95.2)
- added R27: 1k, Resistor_THT:R_Axial_DIN0207_L6.3mm_D2.5mm_P7.62mm_Horizontal, F.Cu at (22.9, 85.1)
- added R28: 4.7k, Resistor_THT:R_Axial_DIN0207_L6.3mm_D2.5mm_P7.62mm_Horizontal, F.Cu at (29.2, 102.9)
- added R29: 1k, Resistor_THT:R_Axial_DIN0207_L6.3mm_D2.5mm_P7.62mm_Horizontal, F.Cu at (22.9, 61.0)
- added R30: 4.7k, Resistor_THT:R_Axial_DIN0207_L6.3mm_D2.5mm_P7.62mm_Horizontal, F.Cu at (22.9, 73.7)
- moved J6 16.6 mm to (83.8, 69.8)
- moved R15 8.98 mm to (76.2, 87.6), turned to 90 degrees
- moved R18 8.98 mm to (66.0, 73.7)
- moved J7 1.27 mm to (81.3, 54.6)
Connections:
- J1 pad 29: unconnected-(J1-Pad29) -> Net-(J1-Pad29)
- J1 pad 31: unconnected-(J1-Pad31) -> Net-(J1-Pad31)
- U5 pad 4: Net-(U4-Pad5) -> -12V
- U5 pad 8: +5V -> +12V
Routing:
- net Net-(J1-Pad29): track 0.00 -> 135.0 mm
- net Net-(J1-Pad31): track 0.00 -> 105.9 mm
- net +5V: track 79.2 -> 155.7 mm
- net Net-(Q4-Pad1): track 0.00 -> 45.4 mm
- net Net-(U4-Pad5): track 35.3 -> 0.00 mm
- net GND: track 349.8 -> 380.2 mm
- net +12V: track 0.00 -> 25.6 mm
- net Net-(Q4-Pad2): track 0.00 -> 25.2 mm
- net Net-(R15-Pad2): track 94.0 -> 71.0 mm
- net Net-(Q3-Pad1): track 0.00 -> 23.0 mm
- net -12V: track 0.00 -> 19.9 mm
- net Net-(J6-PadT): track 42.8 -> 28.7 mm
- net Net-(J10-PadT): track 0.00 -> 12.0 mm
- net Net-(J9-PadT): track 0.00 -> 10.5 mm
- net Net-(Q3-Pad2): track 0.00 -> 10.3 mm
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Other:
- board size 106.7 x 55.9 mm -> 125.7 x 55.9 mm
- board text added: "GATE OUT 1"
- board text added: "GATE OUT 2"
